File: hw/sch_pcb/USBPDSINK01.kicad_pcb (KiCad board)
At the start: 2 copper layers, 45.5 x 52.9 mm, 53 parts, among them J1 USBC_USB4105-GF-A, J2 HEADER_2x05_PARALLEL, J3 HEADER_2x04_PARALLEL, J4 HEADER_2x03_PARALLEL, J5 HEADER_2x01, J6 HEADER_2x07_PARALLEL, J7 WAGO_2604-3102, M1 HOLE, M2 HOLE, M3 HOLE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

Commit message: Solve some issues form 01A
Parts:
- R4: value R10 -> 10R
- moved FID1 0.14 mm to (134.7, 105.5)
Connections:
- J2 pad 5: GND -> /EXT_PWR
- J2 pad 6: GND -> /EXT_PWR
- J4 pad 3: GND -> /EXT_PWR
- J4 pad 4: GND -> /EXT_PWR
- JP3 pad 3: GND -> /EXT_PWR
Routing:
- net /EXT_PWR: track 0.00 -> 23.9 mm
- net GND: track 25.6 -> 18.3 mm, vias 14 -> 13
- net VCC: track 91.5 -> 96.5 mm
- net /PWR_OK3: track 29.2 -> 27.8 mm
- net Net-(D1-A): track 3.58 -> 4.66 mm
- net Net-(D5-A): track 7.65 -> 8.30 mm
- net /PWR_OK2: track 31.3 -> 31.9 mm
Other:
- rule pad_to_mask_clearance: 0.2 -> 0.15
