File: hw/sch_pcb/USBPDSINK01.kicad_sch (KiCad schematic)
At the start: 53 parts, among them J1 USBC_USB4105-GF-A, J11 WAGO_2604-3102, J2 HEADER_2x05_PARALLEL, J3 HEADER_2x04_PARALLEL, J4 HEADER_2x03_PARALLEL, J5 HEADER_2x01, J6 HEADER_2x07_PARALLEL, M1 HOLE, M2 HOLE, M3 HOLE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

Commit message: add ustid, change LDO
Parts:
- C1, C2, C7, C8: UST_ID (none) -> 5c70984712875079b91f8b50
- C4: UST_ID (none) -> 5c70984712875079b91f8b4c
- C5, C6: UST_ID (none) -> 5c70984712875079b91f8b53
- D1, D4: UST_ID (none) -> 64ab2fba76c82a1d3b57877d
- D2: UST_ID (none) -> 650b4b13462c6d9e7205456a
- D3: UST_ID (none) -> 650b4b9e462c6d9e7205459d
- D5: UST_ID (none) -> 64ab2ec176c82a1d3b57875b
- R1, R10, R22: UST_ID (none) -> 639ed3d540d28a66c9e88a9e
- R11: UST_ID (none) -> 5c70984512875079b91f8977
- R12: UST_ID (none) -> 5c70984612875079b91f89a3
- R13, R14, R15, R16, R17, R18, R19, R20, R21: UST_ID (none) -> 5c70984612875079b91f8995
- R3, R5, R6: value 65R -> 62R; MFPN R0805 65R 1% -> R0805 62R 1%; MPN R0805 65R 1% -> R0805 62R 1%; UST_ID (none) -> 5c70984512875079b91f8974
- R4: UST_ID (none) -> 5c70984512875079b91f896d
- R7: value 60R -> 62R; MFPN R0805 60R 1% -> R0805 62R 1%; MPN R0805 60R 1% -> R0805 62R 1%; UST_ID (none) -> 5c70984512875079b91f8974
- R8, R9: UST_ID (none) -> 5c70984512875079b91f898c
- U2: value NCP1117-3.3 -> NCV4274CST33T3G; symbol Regulator_Linear:NCP1117-3.3_SOT223 -> Regulator_Linear:LM2936-3.3; MFPN NCP1117DT33G -> NCV4274CST33T3G; MPN NCP1117DT33G -> NCV4274CST33T3G; UST_ID 5c70984712875079b91f8af9 -> 650b45d7462c6d9e720544df
Connections:
- net +3V3: now also U2.3 (VO); no longer U2.2 (VO)
- net GND: now also U2.2 (GND); no longer U2.1 (GND)
- net VBUS: now also U2.1 (VI); no longer U2.3 (VI)

Commit message: Kontrola a priprava PCB na vyrobu
Parts:
- R4: value R10 -> 10R
Changed lines of the file:
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@@
   (symbol (lib_id "Device:R_Small") (at 144.78 162.56 0) (unit 1)
     (in_bom yes) (on_board yes) (dnp no) (fields_autoplaced)
-    (property "Reference" "R4" (at 147.32 161.29 0)
+    (property "Reference" "R4" (at 146.2786 161.536 0)
       (effects (font (size 1.27 1.27)) (justify left))
     )
-    (property "Value" "R10" (at 147.32 163.83 0)
+    (property "Value" "10R" (at 146.2786 163.584 0)
       (effects (font (size 1.27 1.27)) (justify left))
     )

Commit message: Solve some issues form 01A
Connections:
- net GND: no longer J2.5, J2.6, J4.3, J4.4, JP3.3 (B)
- new net EXT_PWR: J2.5, J2.6, J4.3, J4.4, JP3.3 (B)
Changed lines of the file:
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@@
   (junction (at 133.35 160.02) (diameter 0) (color 0 0 0 0)
   )
-  (junction (at 238.76 76.2) (diameter 0) (color 0 0 0 0)
-  )
   (junction (at 26.67 166.37) (diameter 0) (color 0 0 0 0)
   )
@@
   (junction (at 186.69 45.72) (diameter 0) (color 0 0 0 0)
   )
-  (junction (at 238.76 78.74) (diameter 0) (color 0 0 0 0)
+  (junction (at 237.49 78.74) (diameter 0) (color 0 0 0 0)
   )
   (junction (at 246.38 146.05) (diameter 0) (color 0 0 0 0)
@@
     (stroke (width 0) (type default))
   )
-  (wire (pts (xy 238.76 73.66) (xy 238.76 76.2))
-    (stroke (width 0) (type default))
-  )
   (wire (pts (xy 158.75 55.88) (xy 168.91 55.88))
     (stroke (width 0) (type default))
@@
     (stroke (width 0) (type default))
   )
+  (wire (pts (xy 237.49 73.66) (xy 238.76 73.66))
+    (stroke (width 0) (type default))
+  )
   (wire (pts (xy 248.92 35.56) (xy 254 35.56))
     (stroke (width 0) (type default))
@@
     (stroke (width 0) (type default))
   )
-  (wire (pts (xy 238.76 76.2) (xy 238.76 78.74))
+  (wire (pts (xy 237.49 73.66) (xy 237.49 78.74))
+    (stroke (width 0) (type default))
+  )
+  (wire (pts (xy 237.49 78.74) (xy 238.76 78.74))
     (stroke (width 0) (type default))
   )
@@
     )
   )
-  (symbol (lib_id "power:GND") (at 238.76 78.74 0) (unit 1)
+  (symbol (lib_id "power:GND") (at 237.49 78.74 0) (unit 1)
     (in_bom yes) (on_board yes) (dnp no)
-    (property "Reference" "#PWR015" (at 238.76 85.09 0)
-      (effects (font (size 1.27 1.27)) hide)
-    )
-    (property "Value" "GND" (at 242.57 81.28 0)
+    (property "Reference" "#PWR015" (at 237.49 85.09 0)
+      (effects (font (size 1.27 1.27)) hide)
+    )
+    (property "Value" "GND" (at 241.3 81.28 0)
       (effects (font (size 1.27 1.27)))
     )
-    (property "Footprint" "" (at 238.76 78.74 0)
-      (effects (font (size 1.27 1.27)) hide)
-    )
-    (property "Datasheet" "" (at 238.76 78.74 0)
-      (effects (font (size 1.27 1.27)) hide)
-    )
+    (property "Footprint" "" (at 237.49 78.74 0)
+      (effects (font (size 1.27 1.27)) hide)
+    )
+    (property "Datasheet" "" (at 237.49 78.74 0)
+      (effects (font (size 1.27 1.27)) hide)
+    )
